File: ESP32ProtypeBoard.brd (EAGLE design)
At the start: 55.2 x 54.6 mm, 91 parts, among them IC1 ACT4088US-T, IC2 SI4431BDY, J4 VCC_TERMINAL, Q4 BSS138, U1 3.3V, U2 ESP-WROOM-32

Commit message: 3v3 trace extended to left
Routing:
- net +3V3: track 38.8 -> 51.2 mm
- net GND: track 31.0 -> 32.7 mm, vias 31 -> 32
Changed lines of the file:
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@@
 <wire x1="36.195" y1="40.005" x2="38.735" y2="40.005" width="0.2032" layer="16"/>
 <via x="24.892" y="38.1" extent="1-16" drill="0.35"/>
+<wire x1="39.37" y1="34.163" x2="39.0082" y2="34.5248" width="0.4064" layer="16"/>
+<wire x1="39.0082" y1="34.5248" x2="39.0082" y2="34.53919375" width="0.4064" layer="16"/>
+<wire x1="39.0082" y1="34.53919375" x2="38.47619375" y2="35.0712" width="0.4064" layer="16"/>
+<wire x1="38.47619375" y1="35.0712" x2="38.1" y2="35.0712" width="0.4064" layer="16"/>
+<via x="36.83" y="34.29" extent="1-16" drill="0.35"/>
 <wire x1="125.095" y1="27.305" x2="130.175" y2="42.799" width="0" layer="19" extent="1-1"/>
 <wire x1="104.14" y1="29.21" x2="125.095" y2="27.305" width="0" layer="19" extent="1-1"/>
@@
 <via x="43.18" y="41.91" extent="1-16" drill="0.35"/>
 <wire x1="43.18" y1="41.91" x2="43.672" y2="41.91" width="0.2032" layer="1"/>
+<wire x1="43.688" y1="36.195" x2="43.0032" y2="35.5102" width="0.8128" layer="16"/>
+<wire x1="39.87013125" y1="35.5102" x2="39.468165625" y2="35.912165625" width="0.8128" layer="16"/>
+<wire x1="43.0032" y1="35.5102" x2="39.87013125" y2="35.5102" width="0.8128" layer="16"/>
+<wire x1="39.468165625" y1="35.912165625" x2="34.007165625" y2="35.912165625" width="0.8128" layer="16"/>
+<wire x1="34.007165625" y1="35.912165625" x2="32.385" y2="34.29" width="0.8128" layer="16"/>
 <wire x1="109.855" y1="9.525" x2="125.095" y2="29.845" width="0" layer="19" extent="1-1"/>
 <wire x1="88.265" y1="35.245" x2="109.855" y2="9.525" width="0" layer="19" extent="16-16"/>
@@
 <wire x1="38.22929375" y1="32.893" x2="39.44409375" y2="31.6782" width="0.2032" layer="16"/>
 <wire x1="41.2724875" y1="31.6782" x2="39.44409375" y2="31.6782" width="0.2032" layer="16"/>
-<via x="47.371" y="33.274" extent="1-16" drill="0.35"/>
-<wire x1="47.371" y1="33.274" x2="42.8682875" y2="33.274" width="0.2032" layer="16"/>
-<wire x1="42.8682875" y1="33.274" x2="41.2724875" y2="31.6782" width="0.2032" layer="16"/>
-<wire x1="47.371" y1="33.274" x2="47.0516" y2="33.5934" width="0.2032" layer="1"/>
+<via x="47.371" y="33.147" extent="1-16" drill="0.35"/>
+<wire x1="47.371" y1="33.147" x2="42.7412875" y2="33.147" width="0.2032" layer="16"/>
+<wire x1="42.7412875" y1="33.147" x2="41.2724875" y2="31.6782" width="0.2032" layer="16"/>
+<wire x1="47.371" y1="33.147" x2="47.0516" y2="33.4664" width="0.2032" layer="1"/>
 <wire x1="47.0436" y1="41.29" x2="47.0516" y2="41.282" width="0.2032" layer="1"/>
 <wire x1="47.0436" y1="41.29" x2="47.0516" y2="41.298" width="0.2032" layer="1"/>
@@
 <wire x1="47.0516" y1="41.298" x2="47.0516" y2="42.0909875" width="0.2032" layer="1"/>
 <wire x1="47.878" y1="43.689" x2="47.117" y2="44.45" width="0.2032" layer="1"/>
-<wire x1="47.0516" y1="41.282" x2="47.0516" y2="33.5934" width="0.2032" layer="1"/>
+<wire x1="47.0516" y1="41.282" x2="47.0516" y2="33.4664" width="0.2032" layer="1"/>
 <wire x1="47.117" y1="44.45" x2="74.295" y2="40.64" width="0" layer="19" extent="1-1"/>
 </signal>
@@
 <wire x1="61.91" y1="35.56" x2="62.865" y2="34.605" width="0.2032" layer="16"/>
 <wire x1="62.865" y1="34.605" x2="62.865" y2="32.131" width="0.2032" layer="16"/>
-<wire x1="40.64" y1="34.163" x2="41.324" y2="34.847" width="0.2032" layer="16"/>
-<wire x1="41.324" y1="34.847" x2="52.705" y2="34.847" width="0.2032" layer="16"/>
+<wire x1="40.64" y1="34.163" x2="41.197" y2="34.72" width="0.2032" layer="16"/>
+<wire x1="41.197" y1="34.72" x2="52.578" y2="34.72" width="0.2032" layer="16"/>
 <wire x1="76.2" y1="34.925" x2="77.055" y2="48.26" width="0" layer="19" extent="1-1"/>
 <wire x1="64.495" y1="30.495" x2="76.2" y2="34.925" width="0" layer="19" extent="1-1"/>
-<wire x1="52.705" y1="34.847" x2="61.91" y2="35.56" width="0" layer="19" extent="16-16"/>
+<wire x1="52.578" y1="34.72" x2="61.91" y2="35.56" width="0" layer="19" extent="16-16"/>
 </signal>
 <signal name="IO34">
@@
 <wire x1="39.37229375" y1="32.893" x2="40.17889375" y2="32.0864" width="0.2032" layer="16"/>
 <wire x1="40.17889375" y1="32.0864" x2="41.1034" y2="32.0864" width="0.2032" layer="16"/>
-<wire x1="41.1034" y1="32.0864" x2="43.0476" y2="34.0306" width="0.2032" layer="16"/>
-<wire x1="43.0476" y1="34.0306" x2="52.705" y2="34.0306" width="0.2032" layer="16"/>
-<wire x1="52.705" y1="34.0306" x2="60.01" y2="46.99" width="0" layer="19" extent="16-16"/>
+<wire x1="41.1034" y1="32.0864" x2="42.9206" y2="33.9036" width="0.2032" layer="16"/>
+<wire x1="42.9206" y1="33.9036" x2="52.324" y2="33.9036" width="0.2032" layer="16"/>
+<wire x1="52.324" y1="33.9036" x2="60.01" y2="46.99" width="0" layer="19" extent="16-16"/>
 </signal>
 <signal name="PROG_RXD">
@@
 <wire x1="61.91" y1="38.1" x2="60.01" y2="40" width="0.2032" layer="16"/>
 <wire x1="60.01" y1="40" x2="60.01" y2="44.45" width="0.2032" layer="16"/>
-<wire x1="40.64" y1="32.893" x2="41.9735" y2="34.2265" width="0.2032" layer="16"/>
-<wire x1="41.9735" y1="34.2265" x2="42.037" y2="34.29" width="0.2032" layer="16"/>
-<wire x1="42.037" y1="34.29" x2="42.1858" y2="34.4388" width="0.2032" layer="16"/>
-<wire x1="42.1858" y1="34.4388" x2="52.8740875" y2="34.4388" width="0.2032" layer="16"/>
-<wire x1="52.8740875" y1="34.4388" x2="61.91" y2="38.1" width="0" layer="19" extent="16-16"/>
+<wire x1="40.64" y1="32.893" x2="42.0588" y2="34.3118" width="0.2032" layer="16"/>
+<wire x1="42.0588" y1="34.3118" x2="52.7470875" y2="34.3118" width="0.2032" layer="16"/>
+<wire x1="52.7470875" y1="34.3118" x2="61.91" y2="38.1" width="0" layer="19" extent="16-16"/>
 </signal>
 <signal name="+12V">
